Commit message: display urdf model

File: src/vehicle_chassis/vehicle_description/urdf/pavs.urdf (robot description, URDF)
Before this commit: robot yahboomcar, 9 links, 8 joints
Links:
- link back_left_link: geometry collision mesh filename=package://vehicle_description/meshes/back_right_link.STL; visual mesh filename=package://vehicle_description/meshes/back_right_link.STL
- link back_right_link: geometry collision mesh filename=package://vehicle_description/meshes/back_right_link.STL; visual mesh filename=package://vehicle_description/meshes/back_right_link.STL
- link base_link: geometry collision mesh filename=package://vehicle_description/meshes/base_link.STL; visual mesh filename=package://vehicle_description/meshes/base_link.STL
- link camera_link: geometry collision mesh filename=package://vehicle_description/meshes/camera_link.STL; visual mesh filename=package://vehicle_description/meshes/camera_link.STL
- link front_left_steer: geometry collision mesh filename=package://vehicle_description/meshes/front_left_steer.STL; visual mesh filename=package://vehicle_description/meshes/front_left_steer.STL
- link front_left_wheel: geometry collision mesh filename=package://vehicle_description/meshes/back_right_link.STL; visual mesh filename=package://vehicle_description/meshes/back_right_link.STL
- link front_right_steer: geometry collision mesh filename=package://vehicle_description/meshes/front_left_steer.STL; visual mesh filename=package://vehicle_description/meshes/front_left_steer.STL
- link front_right_wheel: geometry collision mesh filename=package://vehicle_description/meshes/back_right_link.STL; visual mesh filename=package://vehicle_description/meshes/back_right_link.STL
- link laser_link: geometry collision mesh filename=package://vehicle_description/meshes/laser_link.STL; visual mesh filename=package://vehicle_description/meshes/laser_link.STL

File: src/vehicle_chassis/vehicle_description/urdf/pavs.urdf.xacro (robot description, xacro)
@@ -3,5 +3,5 @@
      Commit Version: 1.5.1-0-g916b5db  Build Version: 1.5.7152.31018
      For more information, please see http://wiki.ros.org/sw_urdf_exporter -->
-<robot name="yahboomcar_R2" xmlns:xacro="http://ros.org/wiki/xacro">
+<robot name="pavs" xmlns:xacro="http://ros.org/wiki/xacro">
   <!--xacro:include filename="$(find vehicle_description)/urdf/yahboomcar_R2.gazebo.xacro"/-->
   <link name="imu_link"/>
